Commit message: Filled out URDF in demo134

File: point/urdf/threedofexample.urdf (robot description, URDF)
Before this commit: robot threedofexample, 9 links, 8 joints
Links:
- link baseplate: geometry visual box size=0.2 0.1 0.0230
- link lowerarm: geometry visual mesh filename=package://basic134/meshes/basiclink.stl
- link upperarm: geometry visual box size=0.6 0.08 0.00570
Joints:
- joint elbow: origin xyz=0 0 -0.0311 rpy=3.1415 0 0 -> xyz=0 0 0.0311 rpy=0 0 0
- joint lbracket: origin xyz=0.03 0 0.11317 rpy=0 -1.5708 0 -> xyz=0 0.1 0.11337 rpy=0 -1.5708 1.5708
- joint lowerarm: origin xyz=0.366 0 0.00285 rpy=0 0 0 -> xyz=0.5 0 0.00285 rpy=0 0 0
- joint upperarm: origin xyz=0.4085 0 0.0057 rpy=0 0 0 -> xyz=0.5 0 0.0057 rpy=0 0 0

Commit message: Working on demo
Co-authored-by: Edward Speer <espeer@caltech.edu>
Co-authored-by: joroberts777 <joroberts777@users.noreply.github.com>

File: point/urdf/threedofexample.urdf (robot description, URDF)
Before this commit: robot threedofexample, 9 links, 8 joints
Links:
- link baseplate: geometry visual box size=0.2 0.1 0.01235
- link lowerarm: geometry visual box size=0.406 0.08 0.00570
- link upperarm: geometry visual box size=0.454 0.08 0.00570
Joints:
- joint elbow: origin xyz=0 0 0.0311 rpy=0 0 0 -> xyz=0 0 -0.0311 rpy=3.1415 0 0
- joint lbracket: origin xyz=0 0.1 0.11337 rpy=0 -1.5708 1.5708 -> xyz=0.03 0 0.11317 rpy=0 -1.5708 0
- joint lowerarm: origin xyz=0.5 0 0.00285 rpy=0 0 0 -> xyz=0.366 0 0.00285 rpy=0 0 0
- joint upperarm: origin xyz=0.5 0 0.0057 rpy=0 0 0 -> xyz=0.4085 0 0.0057 rpy=0 0 0
