Commit message: WIP 1_18

File: basic134/urdf/threedofexample.urdf (robot description, URDF)
Before this commit: robot threedofexample, 9 links, 8 joints
Joints:
- joint elbow: origin xyz=0 0 -0.0311 rpy=3.1415 0 0 -> xyz=0 0 0.035 rpy=0 0 3.14159
- joint lowerarm: origin xyz=0.366 0 0.00285 rpy=0 0 0 -> xyz=-0.366 0 0.00285 rpy=0 0 0
- joint upperarm: origin xyz=0.4085 0 0.0057 rpy=0 0 0 -> xyz=0.4085 0 0.0057 rpy=3.14159 0 0

File: point/urdf/threedofexample.urdf (robot description, URDF)
Before this commit: robot threedofexample, 9 links, 8 joints
Joints:
- joint elbow: origin xyz=0 0 -0.0311 rpy=3.1415 0 0 -> xyz=0 0 -0.0311 rpy=0 0 0

Commit message: receives commands from terminal correctly

File: basic134/urdf/threedofexample.urdf (robot description, URDF)
Before this commit: robot threedofexample, 9 links, 8 joints
Joints:
- joint placement: origin xyz=0 0 0 rpy=0 0 0 -> xyz=-0.33 0 0 rpy=0 0 0

Commit message: Calibrate positioning; goals3

File: basic134/urdf/threedofexample.urdf (robot description, URDF)
Before this commit: robot threedofexample, 9 links, 8 joints
Links:
- link baseplate: geometry visual box size=0.2 0.1 0.0125
- link lowerarm: geometry visual mesh filename=package://basic134/meshes/pointer.stl scale=0.001 0.001 0.001
- link upperarm: geometry visual mesh filename=package://basic134/meshes/upperarm.stl scale=0.001 0.001 0.001
Joints:
- joint baseplate: origin xyz=0 0 0.0230 rpy=0 0 -1.5708 -> xyz=0 0.04 0.0125 rpy=0 0 -1.5708
- joint lbracket: origin xyz=0.03 0 0.11317 rpy=0 -1.5708 0 -> xyz=0.03 0 0.11 rpy=0 -1.5708 0
- joint lowerarm: origin xyz=-0.366 0 0.00285 rpy=0 0 0 -> xyz=-0.37 0 0.00285 rpy=0 0 0
- joint upperarm: origin xyz=0.4085 0 0.0057 rpy=3.14159 0 0 -> xyz=0.38 0 0.0057 rpy=3.14159 0 0
